Commit message: my square robot

File: whereami/udacity_bot.xacro (robot description, xacro)
@@ -1,167 +1,232 @@
-<?xml version="1.0"?>
-<robot name="udacity_bot" xmlns:xacro="http://www.ros.org/wiki/xacro">
-<xacro:include filename="$(find udacity_bot)/urdf/udacity_bot.gazebo" />
-  <link name="robot_footprint"></link>
-  <joint name="robot_footprint_joint" type="fixed">
-    <origin xyz="0 0 0" rpy="0 0 0" />
-    <parent link="robot_footprint"/>
-    <child link="chassis" />
-  </joint>
-  <link name="chassis">
-    <pose>0 0 0.1 0 0 0</pose>
-    <inertial>
-      <mass value="15.0"/>
-      <origin xyz="0.0 0 0" rpy=" 0 0 0"/>
-      <inertia
+<?xml version='1.0'?>
+<robot name="udacity_bot"
+	xmlns:xacro="http://www.ros.org/wiki/xacro">
+	<material name="blue">
+		<color rgba="0 0 0.8 1"/>
+	</material>
+	<material name="green">
+		<color rgba="0 1 0 1"/>
+	</material>
+	<xacro:include filename="$(find udacity_bot)/urdf/udacity_bot.gazebo" />
+	<link name="robot_footprint"></link>
+	<joint name="robot_footprint_joint" type="fixed">
+		<origin xyz="0 0 0" rpy="0 0 0" />
+		<parent link="robot_footprint"/>
+		<child link="chassis" />
+	</joint>
+<link name="chassis">
+		<inertial>
+			<mass value="15.0"/>
+			<origin xyz="0.0 0 0" rpy=" 0 0 0"/>
+			<inertia
           ixx="0.1" ixy="0" ixz="0"
           iyy="0.1" iyz="0"
           izz="0.1"
       />
-    </inertial>
-    <collision name="collision">
-      <origin xyz="0 0 0" rpy=" 0 0 0"/>
-      <geometry>
-        <box size=".4 .2 .1"/>
-      </geometry>
-    </collision>
-    <visual name="chassis_visual">
-      <origin xyz="0 0 0" rpy=" 0 0 0"/>
-      <geometry>
-        <box size=".4 .2 .1"/>
-      </geometry>
-     </visual>
-    <collision name="back_caster_collision">
-      <origin xyz="-0.15 0 -0.05" rpy=" 0 0 0"/>
-      <geometry>
-        <sphere radius="0.05"/>
-      </geometry>
-      <surface>
-        <friction>
-          <ode>
-            <mu>0</mu>
-            <mu2>0</mu2>
-            <slip1>1.0</slip1>
-            <slip2>1.0</slip2>
-          </ode>
-        </friction>
-      </surface>
-    </collision>
-    <visual name="back_caster_visual">
-      <origin xyz="-0.15 0 -0.05" rpy=" 0 0 0"/>
-      <geometry>
-        <sphere radius="0.05"/>
-      </geometry>
-    </visual>
-    <collision name="front_caster_collision">
-      <origin xyz="0.15 0 -0.05" rpy=" 0 0 0"/>
-      <geometry>
-        <sphere radius="0.05"/>
-      </geometry>
-      <surface>
-        <friction>
-          <ode>
-            <mu>0</mu>
-            <mu2>0</mu2>
-            <slip1>1.0</slip1>
-            <slip2>1.0</slip2>
-          </ode>
-        </friction>
-      </surface>
-    </collision>
-    <visual name="front_caster_visual">
-      <origin xyz="0.15 0 -0.05" rpy=" 0 0 0"/>
-      <geometry>
-        <sphere radius="0.05"/>
-      </geometry>
-    </visual>
-  </link>
-<link name="left_wheel">
-    <collision name="collision">
-	 	<origin xyz="0 0 0" rpy="0 1.5707 1.5707"/>
-          <geometry>
-            <cylinder length="0.05" radius="0.1"/>
-          </geometry>
-        </collision>
-        <visual name="visual">
-	<origin xyz="0 0 0" rpy="0 1.5707 1.5707"/>
-          <geometry>
-            <cylinder length="0.05" radius="0.1"/>
-          </geometry>
-        </visual>
-	<inertial>
-     <origin xyz="0 0 0" rpy="0 1.5707 1.5707"/>
-     <mass value="5"/>
-     <inertia ixx=".1"  ixy="0"  ixz="0" iyy=".1" iyz="0" izz=".1" />
-   </inertial>
- </link>
-  <joint type="continuous" name="left_wheel_hinge">
-    <origin xyz="0 0.15 0" rpy="0 0 0"/>
-    <child link="left_wheel"/>
-    <parent link="chassis"/>
-    <axis xyz="0 1 0" />
-    <limit effort="10000" velocity="1000"/>
-    <joint_properties damping="1.0" friction="1.0"/>
-  </joint>
-<link name="right_wheel">
-    <collision name="collision">
-	 	<origin xyz="0 0 0" rpy="0 1.5707 1.5707"/>
-          <geometry>
-            <cylinder length="0.05" radius="0.1"/>
-          </geometry>
-        </collision>
-        <visual name="visual">
-	<origin xyz="0 0 0" rpy="0 1.5707 1.5707"/>
-          <geometry>
-            <cylinder length="0.05" radius="0.1"/>
-          </geometry>
-        </visual>
-	<inertial>
-     <origin xyz="0 0 0" rpy="0 1.5707 1.5707"/>
-     <mass value="5"/>
-     <inertia ixx=".1"  ixy="0"  ixz="0" iyy=".1" iyz="0" izz=".1" />
-   </inertial>
- </link>
-  <joint type="continuous" name="right_wheel_hinge">
-    <origin xyz="0 -0.15 0" rpy="0 0 0"/>
-    <child link="right_wheel"/>
-    <parent link="chassis"/>
-    <axis xyz="0 1 0" />
-    <limit effort="10000" velocity="1000"/>
-    <joint_properties damping="1.0" friction="1.0"/>
-  </joint>
-<link name ="camera">
-<origin xyz="0 0 0" rpy="0 0 0"/>
-<visual>
-<origin xyz=".20 0 0" rpy="0 0 0"/>
-<geometry>
-<box size="0.05 0.03 0.03"/>
-</geometry>
-</visual>
-<inertial>
-     <mass value=".1"/>
-     <inertia ixx="1e-6"  ixy="0"  ixz="0" iyy="1e-6" iyz="0" izz="1e-6"/>
- </inertial>
-</link>
-<joint type="fixed" name="camera_joint">
-<orign xyz="0.2 0 0" rpy="0 0 0"/>
-<child link="camera"/>
-<parent link="chassis"/>
-</joint>
-<link name="hokuyo">
-<origin xyz="0 0 0" rpy="0 0 0"/>
-<visual>
-<geometry>
- <mesh filename="package://udacity_bot/meshes/hokuyo.dae"/>
-</geometry>
-</visual>
-<inertial>
-     <mass value=".1"/>
-     <inertia ixx="1e-6"  ixy="0"  ixz="0" iyy="1e-6" iyz="0" izz="1e-6"/>
- </inertial>
-</link>
-<joint type="fixed" name="hokuyo_joint">
-<origin xyz="0.15 0 0.1" rpy="0 0 0"/>
-<child link="hokuyo"/>
-<parent link="chassis"/>
-</joint>
+		</inertial>
+		<collision name='collision'>
+			<origin xyz="0 0 0" rpy=" 0 0 0"/>
+			<geometry>
+				 <box size="0.4 0.4 0.1"/>
+				<!-- <cylinder length="0.1" radius="0.3"/> -->
+			</geometry>
+		</collision>
+		<visual>
+			<geometry>
+				 <box size="0.4 0.4 0.1"/>
+				<!-- <cylinder length="0.1" radius="0.3"/>-->
+			</geometry>
+			<origin rpy="0 0 0" xyz="0 0 0"/>
+			<material name="blue"/>
+		</visual>
+	<visual name='left_caster_visual'>
+			<origin xyz="0.15 -0.15 -0.05" rpy=" 0 0 0"/>
+			<geometry>
+				<sphere radius="0.04"/>
+			</geometry>
+			<material name="white"/>
+		</visual>
+		<collision name='left_caster_collision'>
+			<origin xyz="0.15 -0.15 -0.05" rpy=" 0 0 0"/>
+			<geometry>
+				<sphere radius="0.05"/>
+			</geometry>
+			<surface>
+				<friction>
+					<ode>
+						<mu>0</mu>
+						<mu2>0</mu2>
+						<slip1>1.0</slip1>
+						<slip2>1.0</slip2>
+					</ode>
+				</friction>
+			</surface>
+		</collision>
+		<visual name='right_caster_visual'>
+			<origin xyz="-0.15 0.15 -0.05" rpy=" 0 0 0"/>
+			<geometry>
+				<sphere radius="0.04"/>
+			</geometry>
+			<material name="white"/>
+		</visual>
+		<collision name='right_caster_collision'>
+			<origin xyz="-0.15 0.15 -0.05" rpy=" 0 0 0"/>
+			<geometry>
+				<sphere radius="0.05"/>
+			</geometry>
+			<surface>
+				<friction>
+					<ode>
+						<mu>0</mu>
+						<mu2>0</mu2>
+						<slip1>1.0</slip1>
+						<slip2>1.0</slip2>
+					</ode>
+				</friction>
+			</surface>
+		</collision>
+		<visual name='back_caster_visual'>
+			<origin xyz="-0.15 -0.15 -0.05" rpy=" 0 0 0"/>
+			<geometry>
+				<sphere radius="0.04"/>
+			</geometry>
+			<material name="white"/>
+		</visual>
+		<collision name='back_caster_collision'>
+			<origin xyz="-0.15 -0.15 -0.05" rpy=" 0 0 0"/>
+			<geometry>
+				<sphere radius="0.05"/>
+			</geometry>
+			<surface>
+				<friction>
+					<ode>
+						<mu>0</mu>
+						<mu2>0</mu2>
+						<slip1>1.0</slip1>
+						<slip2>1.0</slip2>
+					</ode>
+				</friction>
+			</surface>
+		</collision>
+		<visual name='front_caster_visual'>
+			<origin xyz="0.15 0.15 -0.05" rpy=" 0 0 0"/>
+			<geometry>
+				<sphere radius="0.04"/>
+			</geometry>
+			<material name="white"/>
+		</visual>
+		<collision name='front_caster_collision'>
+			<origin xyz="0.15 0.15 -0.05" rpy=" 0 0 0"/>
+			<geometry>
+				<sphere radius="0.05"/>
+			</geometry>
+			<surface>
+				<friction>
+					<ode>
+						<mu>0</mu>
+						<mu2>0</mu2>
+						<slip1>1.0</slip1>
+						<slip2>1.0</slip2>
+					</ode>
+				</friction>
+			</surface>
+		</collision>
+	</link>
+	<link name="left_wheel">
+		<visual>
+			<geometry>
+				<cylinder length="0.05" radius="0.06"/>
+			</geometry>
+			<origin rpy="0 1.5707 1.5707" xyz="0 0 0"/>
+			<material name="green"/>
+		</visual>
+		<collision name="collision">
+			<origin xyz="0 0 0" rpy="0 1.5707 1.5707"/>
+			<geometry>
+				<cylinder length="0.05" radius="0.1"/>
+			</geometry>
+		</collision>
+		<inertial>
+			<origin xyz="0 0 0" rpy="0 1.5707 1.5707"/>
+			<mass value="5"/>
+			<inertia ixx=".1"  ixy="0"  ixz="0" iyy=".1" iyz="0" izz=".1" />
+		</inertial>
+	</link>
+	<joint name="left_wheel_hinge" type="continuous">
+		<parent link="chassis"/>
+		<child link="left_wheel"/>
+		<origin xyz="0 0.25 0" rpy="0 0 0"/>
+	</joint>
+	<link name="right_wheel">
+		<visual>
+			<geometry>
+				<cylinder length="0.05" radius="0.06"/>
+			</geometry>
+			<origin rpy="0 1.5707 1.5707" xyz="0 0 0"/>
+			<material name="green"/>
+		</visual>
+		<collision name="collision">
+			<origin xyz="0 0 0" rpy="0 1.5707 1.5707"/>
+			<geometry>
+				<cylinder length="0.05" radius="0.1"/>
+			</geometry>
+		</collision>
+		<inertial>
+			<origin xyz="0 0 0" rpy="0 1.5707 1.5707"/>
+			<mass value="5"/>
+			<inertia ixx=".1"  ixy="0"  ixz="0" iyy=".1" iyz="0" izz=".1" />
+		</inertial>
+	</link>
+	<joint name="right_wheel_hinge" type="continuous">
+		<parent link="chassis"/>
+		<child link="right_wheel"/>
+		<origin xyz="0 -0.25 0" rpy="0 0 0"/>
+	</joint>
+	<link name ="camera">
+		<origin xyz="0 0 0" rpy="0 0 0"/>
+		<collision>
+			<origin xyz="0.2 0 0" rpy="0 0 0"/>
+			<geometry>
+				<box size="0.05 0.05 0.05"/>
+			</geometry>
+		</collision>
+		<visual>
+			<origin xyz=".20 0 0" rpy="0 0 0"/>
+			<geometry>
+				<box size="0.05 0.05 0.05"/>
+			</geometry>
+		</visual>
+		<inertial>
+			<mass value="0.1"/>
+			<inertia ixx="1e-6"  ixy="0"  ixz="0" iyy="1e-6" iyz="0" izz="1e-6"/>
+		</inertial>
+	</link>
+	<joint type="fixed" name="camera_joint">
+		<orign xyz="0.2 0 0" rpy="0 0 0"/>
+		<child link="camera"/>
+		<parent link="chassis"/>
+	</joint>
+	<link name="hokuyo">
+		<origin xyz="0 0 0" rpy="0 0 0"/>
+		<collision name="collision">
+			<origin xyz="0 0 0" rpy="0 1.5707 1.5707"/>
+			<geometry>
+				<box size="0.1 0 0"/>
+			</geometry>
+		</collision>
+		<visual>
+			<geometry>
+				<mesh filename="package://udacity_bot/meshes/hokuyo.dae"/>
+			</geometry>
+		</visual>
+		<inertial>
+			<mass value=".1"/>
+			<inertia ixx="1e-6"  ixy="0"  ixz="0" iyy="1e-6" iyz="0" izz="1e-6"/>
+		</inertial>
+	</link>
+	<joint type="fixed" name="hokuyo_joint">
+		<origin xyz="0.15 0 0.1" rpy="0 0 0"/>
+		<child link="hokuyo"/>
+		<parent link="chassis"/>
+	</joint>
 </robot>
